Commit message: feat: tilt iris_rgb camera downward
upward racing tilt was showing mostly sky during low speed tests

File: src/sitl_launcher/urdf/iris_rgb.urdf (robot description, URDF)
Before this commit: robot iris, 4 links, 3 joints
Joints:
- joint camera_joint: origin xyz=0.135 0 0 rpy=0 -0.26 0 -> xyz=0.135 0 0 rpy=0 0.3491 0
